File: hardware/CLN17/V2.0/CLN17-V2.0.kicad_sch (KiCad schematic)
At the start: 88 parts, among them IC1 STM32G431CB, J1 PWR, J2 PWR, J3 TYPE-C-31-M-12, J4 Motor, J5 CTRL, J6 CAN, J7 CAN, J8 DEBUG, J9 IO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

Commit message: [WIP] Before adding CAN connectors
Parts:
- removed J9: IO, FP_lib:2x2P2.00mm_Vertical_SMD, symbol Connector_Generic:Conn_02x02_Odd_Even
- removed Q1: AO3401, FP_lib:SOT-23-3, symbol Transistor_FET:AO3401A
- removed R17, R18, R19, R35: 120, FP_lib:R0402, symbol R_Small
- removed R20, R21, R22, R27: 5.1k, FP_lib:R0402, symbol R_Small
- removed R32: 10k, FP_lib:R0402, symbol R_Small
- removed R33: 510, FP_lib:R0402, symbol R_Small
- added J10: CAN_OUT, FP_lib:PH2.0 4P, symbol Conn_01x04
- added J9: CAN_IN, FP_lib:PH2.0 4P, symbol Conn_01x04
- U10, U5: footprint footprints:DFN-2510 -> FP_lib:DFN-2510
Connections:
- net _DIR is gone; now on net CTRL_MISO: R1.1, U10.4 (I/O3), U10.7 (I/O3)
- net _ENB is gone; now on net CTRL_MOSI: R26.1, U10.5 (I/O4), U10.6 (I/O4)
- net _ERR is gone; now on net CTRL_SCK: R3.1, U10.2 (I/O2), U10.9 (I/O2)
- net _STP is gone; now on net CTRL_CS: R2.1, U10.1 (I/O1), U10.10
- net DIR: no longer names the net of J5.3 (Pin_3), R1.2
- net ENB: no longer names the net of J5.2 (Pin_2), R26.2
- net ERR: no longer names the net of J5.5 (Pin_5), R3.2
- net STP: no longer names the net of J5.4 (Pin_4), R2.2
Other:
- note removed: "Control IO PullUp"
- note removed: "Control IO protection"
- note removed: "ENB 5V"
- note removed: "Expansion board connector"
- moved on the sheet: J5, R1, R2, R26, R3, U10

Commit message: [WIP] Before rotating the CAN transceiver
Parts:
- removed J2: PWR, FP_lib:XH2.54 2P, symbol Conn_01x02
- removed J6, J7: CAN, FP_lib:PH2.0 2P, symbol Conn_01x02
Connections:
- net CAN_N: now also J10.1 (Pin_1), J9.1 (Pin_1)
- net CAN_P: now also J10.2 (Pin_2), J9.2 (Pin_2)
- net GND: now also J10.3 (Pin_3), J9.3 (Pin_3)
- net VCON: now also J10.4 (Pin_4), J9.4 (Pin_4)
Other:
- note added: "CAN-Bus And Power Daisy Chain Including Protection"
- note removed: "CAN-Bus Daisy Chain + Protection"
- note removed: "Power Daisy Chain + Protection"
- moved on the sheet: D1, D3, D4, D5, J1, J10, J9

Commit message: Almost done
Parts:
- removed J5: CTRL, FP_lib:PH2.0 5P, symbol Connector_Generic:Conn_01x05
- removed R26: 120, FP_lib:R0402, symbol R_Small
- added J2: AUX, FP_lib:JST-S7B-ZR, symbol Connector_Generic:Conn_01x07
- added R14, R17, R8: 120, FP_lib:R0402, symbol R_Small
- added R18, R19: 1k, FP_lib:R0402, symbol R_Small
Connections:
- net +3V3A: now also R18.1
- net CAN_N: now also J10.2 (Pin_2), J9.2 (Pin_2); no longer J10.1 (Pin_1), J9.1 (Pin_1)
- net CAN_P: now also J10.1 (Pin_1), J9.1 (Pin_1); no longer J10.2 (Pin_2), J9.2 (Pin_2)
- net CTRL_CS: now also R2.2; no longer R2.1, U10.1 (I/O1), U10.10
- net CTRL_MISO: now also R3.2; no longer R1.1, U10.4 (I/O3), U10.7 (I/O3)
- net CTRL_MOSI: now also R8.2; no longer U10.5 (I/O4), U10.6 (I/O4)
- net CTRL_SCK: now also R1.2; no longer R3.1, U10.2 (I/O2), U10.9 (I/O2)
- net EXP_RX: now also R17.2
- net EXP_TX: now also R14.2
- net GND: now also J10.4 (Pin_4), J9.4 (Pin_4), J2.7 (Pin_7), R19.2; no longer J10.3 (Pin_3), J9.3 (Pin_3), U6.5 (REF), U7.5 (REF)
- net VCON: now also J10.3 (Pin_3), J9.3 (Pin_3); no longer J10.4 (Pin_4), J9.4 (Pin_4)
- net ~{CTRL_5V}: no longer names the net of IC1.25 (PB12)
- new net: J2.1 (Pin_1), R1.1, U10.1 (I/O1), U10.10
- new net: J2.2 (Pin_2), R3.1, U10.2 (I/O2), U10.9 (I/O2)
- new net: J2.3 (Pin_3), R8.1, U10.4 (I/O3), U10.7 (I/O3)
- new net: J2.4 (Pin_4), R2.1, U10.5 (I/O4), U10.6 (I/O4)
- new net: J2.5 (Pin_5), R17.1
- new net: J2.6 (Pin_6), R14.1
- new net CURR_REF: R18.2, R19.1, U6.5 (REF), U7.5 (REF)
- no-connect marks 5 -> 6
Other:
- note removed: "1"
- note removed: "2"
- note removed: "3"
- note removed: "4"
- note removed: "5"
- note removed: "5V"
- note removed: "A"
- note removed: "B"
- note removed: "CK"
- note removed: "CS"
- note removed: "DIR"
- note removed: "ENB"
- note removed: "ERR"
- note removed: "GND"
- note removed: "I2C3"
- note removed: "MISO"
- note removed: "MOSI"
- note removed: "RX"
- note removed: "SCK"
- note removed: "SCL"
- note removed: "SDA"
- note removed: "SPI3"
- note removed: "STP"
- note removed: "STP-DIR"
- note removed: "TIM3"
- note removed: "TX"
- note removed: "USART2"
- note removed: "Z"
- moved on the sheet: U10
