File: hardware/CLN17/V2.0/CLN17-V2.0.kicad_pcb (KiCad board)
At the start: 4 copper layers, 38 x 39 mm, 97 parts, among them IC1 STM32G431CB, J1 PWR, J2 PWR, J3 TYPE-C-31-M-12, J4 Motor, J5 CTRL, J6 CAN, J7 CAN, J8 DEBUG, J9 IO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

Commit message: [WIP] Before adding CAN connectors
Parts:
- removed Q1: AO3401, FP_lib:SOT-23-3
- removed R17, R18, R19, R35: 120, FP_lib:R0402
- removed R20, R21, R22, R27: 5.1k, FP_lib:R0402
- removed R32: 10k, FP_lib:R0402
- removed R33: 510, FP_lib:R0402
- added J10: CAN_OUT, FP_lib:PH2.0 4P, F.Cu at (63.2, 38.4)
- J9: value IO -> CAN_IN; footprint FP_lib:2x2P2.00mm_Vertical_SMD -> FP_lib:PH2.0 4P
- U10, U5: footprint footprints:DFN-2510 -> FP_lib:DFN-2510
- moved J9 31.4 mm to (63.2, 30.5), turned to 0 degrees
Connections:
- net /DIR renamed Net-(J5-Pin_3)
- net /ENB renamed Net-(J5-Pin_2)
- net /ERR renamed Net-(J5-Pin_5)
- net /STP renamed Net-(J5-Pin_4)
- J9 pad 1: VBUS -> unconnected-(J9-Pin_1-Pad1)
- J9 pad 2: GND -> unconnected-(J9-Pin_2-Pad2)
- J9 pad 3: /EXP_TX -> unconnected-(J9-Pin_3-Pad3)
- J9 pad 4: /EXP_RX -> unconnected-(J9-Pin_4-Pad4)
- R1 pad 1: /_DIR -> /CTRL_MISO
- R2 pad 1: /_STP -> /CTRL_CS
- R26 pad 1: /_ENB -> /CTRL_MOSI
- R3 pad 1: /_ERR -> /CTRL_SCK
- U10 pad 1: /_STP -> /CTRL_CS
- U10 pad 10: /_STP -> /CTRL_CS
- U10 pad 2: /_ERR -> /CTRL_SCK
- U10 pad 4: /_DIR -> /CTRL_MISO
- U10 pad 5: /_ENB -> /CTRL_MOSI
- U10 pad 6: /_ENB -> /CTRL_MOSI
- U10 pad 7: /_DIR -> /CTRL_MISO
- U10 pad 9: /_ERR -> /CTRL_SCK
Routing:
- net /EXP_TX: track 23.5 -> 6.40 mm, vias 2 -> 1
- net /~{CTRL_5V}: track 15.6 -> 0.72 mm, vias 2 -> 1
- net /EXP_RX: track 19.2 -> 4.68 mm, vias 2 -> 1
- net Net-(J5-Pin_2): track 22.3 -> 13.4 mm, vias 3 -> 1
- net /_STP: track 8.40 -> 0.00 mm
- net /_ENB: track 7.58 -> 0.00 mm
- net /_DIR: track 6.99 -> 0.00 mm
- net /_ERR: track 6.76 -> 0.00 mm
- net +3V3: track 11.3 -> 6.10 mm
- net /B2: track 9.71 -> 4.71 mm
- net /B1: track 7.97 -> 2.97 mm
- net /A2: track 9.71 -> 4.71 mm
- net /A1: track 7.97 -> 2.97 mm
- net /CTRL_MOSI: track 25.7 -> 30.0 mm
- net /CTRL_MISO: track 25.5 -> 29.8 mm
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Other:
- board text removed: "5V CS SCL 5V EN"
- board text removed: "A SI SDA CK DIR"
- board text removed: "B SO RX RX STP"
- board text removed: "ENC SPI I2C URT GND"
- board text removed: "Z SCK TX TX ERR"

Commit message: [WIP] Before rotating the CAN transceiver
Parts:
- removed J2: PWR, FP_lib:XH2.54 2P
- removed J6, J7: CAN, FP_lib:PH2.0 2P
- moved J5 56.3 mm to (71.6, 26.3), turned to 0 degrees
- moved R1 51.4 mm to (72.0, 42.0)
- moved R2 51.4 mm to (72.0, 44.4)
- moved R26 51.4 mm to (72.0, 41.0)
- moved R3 51.4 mm to (72.0, 43.4)
- moved U10 51.4 mm to (73.9, 42.6)
- moved J9 46.5 mm to (16.8, 28.6), turned to 90 degrees
- moved J10 46.4 mm to (16.8, 39.4), turned to 90 degrees
Connections:
- J10 pad 1: unconnected-(J10-Pin_1-Pad1) -> /CAN_N
- J10 pad 2: unconnected-(J10-Pin_2-Pad2) -> /CAN_P
- J10 pad 3: unconnected-(J10-Pin_3-Pad3) -> GND
- J10 pad 4: unconnected-(J10-Pin_4-Pad4) -> VCON
- J9 pad 1: unconnected-(J9-Pin_1-Pad1) -> /CAN_N
- J9 pad 2: unconnected-(J9-Pin_2-Pad2) -> /CAN_P
- J9 pad 3: unconnected-(J9-Pin_3-Pad3) -> GND
- J9 pad 4: unconnected-(J9-Pin_4-Pad4) -> VCON
Routing:
- net Net-(J5-Pin_2): track 13.4 -> 0.00 mm, vias 1 -> 0
- net /CAN_P: track 25.0 -> 13.5 mm, vias 1 -> 2
- net Net-(J5-Pin_3): track 11.5 -> 0.00 mm, vias 1 -> 0
- net /CAN_N: track 24.1 -> 14.3 mm, vias 1 -> 2
- net Net-(J5-Pin_4): track 5.09 -> 0.00 mm, vias 1 -> 0
- net Net-(J5-Pin_5): track 4.96 -> 0.00 mm, vias 1 -> 0
- net /CTRL_CS: track 24.8 -> 21.1 mm
- net /CTRL_MOSI: track 30.0 -> 27.2 mm
- net /CTRL_MISO: track 29.8 -> 27.3 mm
- net GND: track 35.0 -> 32.6 mm, vias 104 -> 103
- net /CTRL_SCK: track 28.3 -> 26.6 mm
Other:
- board text added: "${REFERENCE}"
- board text removed: "L"

Commit message: Almost done
Parts:
- removed J5: CTRL, FP_lib:PH2.0 5P
- removed R26: 120, FP_lib:R0402
- added J2: AUX, FP_lib:JST-S7B-ZR, F.Cu at (50.3, 34.0)
- added R14: 120, FP_lib:R0402, F.Cu at (47.9, 41.8)
- added R17: 120, FP_lib:R0402, F.Cu at (47.9, 40.8)
- added R18: 1k, FP_lib:R0402, F.Cu at (24.9, 32.1)
- added R19: 1k, FP_lib:R0402, F.Cu at (24.9, 33.1)
- added R8: 120, FP_lib:R0402, F.Cu at (47.9, 38.0)
- moved U10 27.1 mm to (47.9, 35.0), turned to -90 degrees
- moved R3 24.5 mm to (47.9, 38.9)
- moved R1 24.2 mm to (47.9, 39.9)
- moved R2 24.1 mm to (47.9, 42.7)
- moved C35 3.25 mm to (27.9, 39.7)
- moved R9 2.78 mm to (23.9, 45.2), turned to 0 degrees
- moved C25 2.40 mm to (23.2, 39.9)
- moved C4 2.18 mm to (45.1, 34.8), turned to 0 degrees
- moved D2 1.96 mm to (21.6, 37.0)
- moved L1 1.84 mm to (24.3, 37.2)
- moved U9 1.84 mm to (22.9, 41.9)
- moved C20 1.61 mm to (27.9, 40.6)
- moved U4 1.61 mm to (29.9, 41.6)
- moved C6 1.23 mm to (47.8, 31.9), turned to 180 degrees
- moved R7 1.16 mm to (23.9, 44.2), turned to 0 degrees
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Connections:
- J10 pad 1: /CAN_N -> /CAN_P
- J10 pad 2: /CAN_P -> /CAN_N
- J10 pad 3: GND -> VCON
- J10 pad 4: VCON -> GND
- J9 pad 1: /CAN_N -> /CAN_P
- J9 pad 2: /CAN_P -> /CAN_N
- J9 pad 3: GND -> VCON
- J9 pad 4: VCON -> GND
- R1 pad 1: /CTRL_MISO -> Net-(J2-Pin_1)
- R1 pad 2: Net-(J5-Pin_3) -> /CTRL_SCK
- R2 pad 1: /CTRL_CS -> Net-(J2-Pin_4)
- R2 pad 2: Net-(J5-Pin_4) -> /CTRL_CS
- R3 pad 1: /CTRL_SCK -> Net-(J2-Pin_2)
- R3 pad 2: Net-(J5-Pin_5) -> /CTRL_MISO
- U10 pad 1: /CTRL_CS -> Net-(J2-Pin_1)
- U10 pad 10: /CTRL_CS -> Net-(J2-Pin_1)
- U10 pad 2: /CTRL_SCK -> Net-(J2-Pin_2)
- U10 pad 4: /CTRL_MISO -> Net-(J2-Pin_3)
- U10 pad 5: /CTRL_MOSI -> Net-(J2-Pin_4)
- U10 pad 6: /CTRL_MOSI -> Net-(J2-Pin_4)
- U10 pad 7: /CTRL_MISO -> Net-(J2-Pin_3)
- U10 pad 9: /CTRL_SCK -> Net-(J2-Pin_2)
- U6 pad 5: GND -> /CURR_REF
- U7 pad 5: GND -> /CURR_REF
Routing:
- net /CURR_REF: track 0.00 -> 26.9 mm, vias 0 -> 2
- net /CAN_P: track 13.5 -> 39.3 mm
- net /CTRL_MISO: track 27.3 -> 1.72 mm, vias 2 -> 0
- net /CTRL_MOSI: track 27.2 -> 1.90 mm, vias 2 -> 0
- net /CAN_N: track 14.3 -> 39.5 mm
- net /CTRL_SCK: track 26.6 -> 1.56 mm, vias 2 -> 0
- net Net-(J2-Pin_4): track 0.00 -> 18.8 mm, vias 0 -> 3
- net GND: track 32.6 -> 48.5 mm, vias 103 -> 105
- net /CTRL_CS: track 21.1 -> 7.32 mm
- net Net-(J2-Pin_3): track 0.00 -> 10.2 mm, vias 0 -> 1
- net Net-(J2-Pin_2): track 0.00 -> 10.0 mm, vias 0 -> 1
- net Net-(J2-Pin_1): track 0.00 -> 8.01 mm
- net /CAN_RX: track 18.5 -> 11.1 mm
- net /CAN_TX: track 19.7 -> 12.9 mm
- net /CAN_SD: track 1.85 -> 7.72 mm
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Other:
- board text removed: "${REFERENCE}"
